Commit message: update vehicle

File: autoVehicle/urdf/autoVehicle.urdf (robot description, URDF)
Before this commit: robot autoVehicle, 5 links, 4 joints
Links:
- added link radar_link, mass 0.014432; collision mesh filename=package://autoVehicle/meshes/radar_link.STL; visual mesh filename=package://autoVehicle/meshes/radar_link.STL
Joints:
- added joint radar_joint: type revolute, parent base_link, child radar_link, origin xyz=0.081864 0.046756 0.061068 rpy=1.5708 0 0, axis 0 1 0, limit lower=0 upper=360 effort=0 velocity=0

Commit message: 首次尝试小车运行。小车仍存在问题。制作了用于测试的世界环境。

File: autoVehicle/urdf/autoVehicle.urdf (robot description, URDF)
Before this commit: robot autoVehicle, 6 links, 5 joints
Links:
- link left_front_wheel: geometry collision cylinder length=0.012 radius=0.0325; visual mesh filename=package://autoVehicle/meshes/left_front_wheel.STL
- link left_rear_wheel: geometry collision cylinder length=0.012 radius=0.0325; visual mesh filename=package://autoVehicle/meshes/left_rear_wheel.STL
- link right_front_wheel: geometry collision cylinder length=0.012 radius=0.0325; visual mesh filename=package://autoVehicle/meshes/right_front_wheel.STL
- link right_rear_wheel: geometry collision cylinder length=0.012 radius=0.0325; visual mesh filename=package://autoVehicle/meshes/right_rear_wheel.STL
Joints:
- joint left_front_joint: axis 1 0 0 -> 0 0 -1
- joint left_rear_joint: axis 0 1 0 -> 0 0 -1
- joint radar_joint: limit lower=0 upper=360 effort=0 velocity=0 -> (none); type revolute -> continuous
- joint right_front_joint: axis 0 1 0 -> 0 0 -1
- joint right_rear_joint: axis 0 1 0 -> 0 0 -1

Commit message: optimize autoVehicle

File: autoVehicle/urdf/autoVehicle.urdf (robot description, URDF)
Before this commit: robot autoVehicle, 6 links, 5 joints
Links:
- link base_link: mass 0.2772 -> 0.446602219201247
- link left_front_wheel: geometry collision mesh filename=package://autoVehicle/meshes/left_front_wheel.STL; visual mesh filename=package://autoVehicle/meshes/left_front_wheel.STL
- link left_rear_wheel: geometry collision mesh filename=package://autoVehicle/meshes/left_rear_wheel.STL; visual mesh filename=package://autoVehicle/meshes/left_rear_wheel.STL
- link right_front_wheel: geometry collision mesh filename=package://autoVehicle/meshes/right_front_wheel.STL; visual mesh filename=package://autoVehicle/meshes/right_front_wheel.STL
- link right_rear_wheel: geometry collision mesh filename=package://autoVehicle/meshes/right_rear_wheel.STL; visual mesh filename=package://autoVehicle/meshes/right_rear_wheel.STL
Joints:
- joint left_front_joint: axis 0 0 -1 -> 0 1 0; origin xyz=0.16516 0.040076 0.018568 rpy=1.5708 0 0 -> xyz=0.07 0.074 -0.012 rpy=0 0 0
- joint left_rear_joint: axis 0 0 -1 -> 0 1 0; origin xyz=0.16745 0.17968 0.018568 rpy=1.5708 0 0 -> xyz=-0.07 0.074 -0.012 rpy=0 0 0
- joint radar_joint: axis 0 1 0 -> 0 0 1; origin xyz=0.081864 0.046756 0.061068 rpy=1.5708 0 0 -> xyz=0.063205 0.015705 0.0305 rpy=0 0 0; type continuous -> fixed
- joint right_front_joint: axis 0 0 -1 -> 0 1 0; origin xyz=-0.0078413 0.039961 0.018568 rpy=1.5708 0 3.1416 -> xyz=0.07 -0.074 -0.012 rpy=0 0 0
- joint right_rear_joint: axis 0 0 -1 -> 0 1 0; origin xyz=-0.0078413 0.17996 0.018568 rpy=1.5708 0 3.1416 -> xyz=-0.07 -0.074 -0.012 rpy=0 0 0
